Commit message: Initial working commit

File: zivid_description/urdf/macros/zivid_one_plus_camera.gazebo.xacro (robot description, xacro)
@@ -2,6 +2,10 @@
 <robot xmlns:xacro="http://www.ros.org/wiki/xacro">
   <xacro:macro name="zivid_one_plus_gazebo" params="prefix">
-    <gazebo reference="camera">
-      <sensor name="camera" type="depth">
+    <!-- <xacro:property name="link_name" value="${prefix}_optical_frame" /> -->
+    <xacro:property name="link_name" value="${prefix}_optical_frame_gazebo" />
+    <xacro:property name="camera_name" value="${prefix}_camera" />
+    <xacro:property name="frame_name" value="${prefix}_optical_frame" />
+    <gazebo reference="${link_name}">
+      <sensor name="${link_name}_camera" type="depth">
         <update_rate>20</update_rate>
         <camera>
@@ -17,29 +21,22 @@
           </clip>
         </camera>
-        <plugin name="camera_plugin" filename="libgazebo_ros_openni_kinect.so">
+        <plugin name="${link_name}_controller" filename="libgazebo_ros_openni_kinect.so">
           <baseline>0.2</baseline>
           <alwaysOn>true</alwaysOn>
-          <!-- Keep this zero, update_rate in the parent <sensor> tag
-            will control the frame rate. -->
-          <updateRate>0.0</updateRate>
-          <cameraName>camera_ir</cameraName>
-          <!--Hardware Driver Topic Names
-              /${prefix}_camera/color/image_color
-              /${prefix}_camera/depth/image
-              /${prefix}_camera/joint_states
-              /${prefix}_camera/points/xyzrgba -->
-          <imageTopicName>/${prefix}_camera/color/image_raw</imageTopicName>
-          <cameraInfoTopicName>/${prefix}_camera/color/camera_info</cameraInfoTopicName>
-          <depthImageTopicName>/${prefix}_camera/depth/image_raw</depthImageTopicName>
-          <depthImageCameraInfoTopicName>/${prefix}_camera/depth/camera_info</depthImageCameraInfoTopicName>
-          <pointCloudTopicName>/${prefix}_camera/depth/points</pointCloudTopicName>
-          <frameName>${prefix}_optical_frame</frameName>
+          <updateRate>1.0</updateRate>
+          <cameraName>${camera_name}_ir</cameraName>
+          <imageTopicName>/${camera_name}/color/image_raw</imageTopicName>
+          <cameraInfoTopicName>/${camera_name}/color/camera_info</cameraInfoTopicName>
+          <depthImageTopicName>/${camera_name}/depth/image_raw</depthImageTopicName>
+          <depthImageInfoTopicName>/${camera_name}/depth/camera_info</depthImageInfoTopicName>
+          <pointCloudTopicName>/${camera_name}/depth/points</pointCloudTopicName>
+          <frameName>${frame_name}</frameName>
           <pointCloudCutoff>0.5</pointCloudCutoff>
           <pointCloudCutoffMax>3.0</pointCloudCutoffMax>
-          <distortionK1>0</distortionK1>
-          <distortionK2>0</distortionK2>
-          <distortionK3>0</distortionK3>
-          <distortionT1>0</distortionT1>
-          <distortionT2>0</distortionT2>
+          <distortionK1>0.00000001</distortionK1>
+          <distortionK2>0.00000001</distortionK2>
+          <distortionK3>0.00000001</distortionK3>
+          <distortionT1>0.00000001</distortionT1>
+          <distortionT2>0.00000001</distortionT2>
           <CxPrime>0</CxPrime>
           <Cx>0</Cx>

File: zivid_description/urdf/macros/zivid_one_plus_camera.xacro (robot description, xacro)
@@ -60,4 +60,12 @@
             <child link="${prefix}_optical_frame"/>
         </joint>
+        <!-- Zivid Optical Frame for Gazebo-->
+        <!-- Unsure why the original code uses y positive out of the sensor rather than x? -->
+        <link name="${prefix}_optical_frame_gazebo"/>
+        <joint name="${prefix}_optical_gazebo_joint" type="fixed">
+            <origin xyz="0.0 0.0 0.0" rpy="${0.5*pi} -${0.5*pi} 0"/>
+            <parent link="${prefix}_optical_frame"/>
+            <child link="${prefix}_optical_frame_gazebo"/>
+        </joint>
         <!--Extensions -->
         <xacro:zivid_one_plus_gazebo prefix="${prefix}"/>
