Commit message: Incorporated underscore outside of prefix

File: zivid_description/urdf/macros/zivid_one_plus_camera.xacro (robot description, xacro)
@@ -15,5 +15,5 @@
     <xacro:macro name="zivid_one_plus_camera" params="prefix type">
         <!-- Zivid Base Link -->
-        <link name="${prefix}base_link">
+        <link name="${prefix}_base_link">
             <!-- Visuals -->
             <visual>
@@ -33,5 +33,5 @@
         </link>
         <!-- Zivid Optical Frame (Measurement Frame)-->
-        <link name="${prefix}optical_frame"/>
+        <link name="${prefix}_optical_frame"/>
         <!-- Set the angle of the optical frame based on the type -->
         <xacro:if value="${type == Zivid_One_Plus_S}" >
@@ -45,8 +45,8 @@
         </xacro:if>
         <!-- Zivid Optical (Measurement) Joint -->
-        <joint name="${prefix}optical_joint" type="fixed">
+        <joint name="${prefix}_optical_joint" type="fixed">
             <origin xyz="0.065 0.062 0.0445" rpy="-${0.5*pi} 0 -${0.5*pi + optical_frame_angle/180*pi}"/>
-            <parent link="${prefix}base_link"/>
-            <child link="${prefix}optical_frame"/>
+            <parent link="${prefix}_base_link"/>
+            <child link="${prefix}_optical_frame"/>
         </joint>
     </xacro:macro>

File: zivid_description/urdf/zivid_one_plus_l_camera.urdf.xacro (robot description, xacro)
@@ -2,4 +2,4 @@
 <robot name="zivid_one_plus_camera_robot" xmlns:xacro="http://www.ros.org/wiki/xacro">
     <xacro:include filename="$(find zivid_description)/urdf/macros/zivid_one_plus_camera.xacro"/>
-    <xacro:zivid_one_plus_camera prefix="zivid_" type="${Zivid_One_Plus_L}"/>
+    <xacro:zivid_one_plus_camera prefix="zivid" type="${Zivid_One_Plus_L}"/>
 </robot>

File: zivid_description/urdf/zivid_one_plus_m_camera.urdf.xacro (robot description, xacro)
@@ -2,4 +2,4 @@
 <robot name="zivid_one_plus_camera_robot" xmlns:xacro="http://www.ros.org/wiki/xacro">
     <xacro:include filename="$(find zivid_description)/urdf/macros/zivid_one_plus_camera.xacro"/>
-    <xacro:zivid_one_plus_camera prefix="zivid_" type="${Zivid_One_Plus_M}"/>
+    <xacro:zivid_one_plus_camera prefix="zivid" type="${Zivid_One_Plus_M}"/>
 </robot>

File: zivid_description/urdf/zivid_one_plus_s_camera.urdf.xacro (robot description, xacro)
@@ -2,4 +2,4 @@
 <robot name="zivid_one_plus_camera_robot" xmlns:xacro="http://www.ros.org/wiki/xacro">
     <xacro:include filename="$(find zivid_description)/urdf/macros/zivid_one_plus_camera.xacro"/>
-    <xacro:zivid_one_plus_camera prefix="zivid_" type="${Zivid_One_Plus_S}"/>
+    <xacro:zivid_one_plus_camera prefix="zivid" type="${Zivid_One_Plus_S}"/>
 </robot>

Commit message: WiP Zivid Simulation

File: zivid_description/urdf/macros/zivid_one_plus_camera.xacro (robot description, xacro)
@@ -1,4 +1,9 @@
 <?xml version="1.0"?>
 <robot xmlns:xacro="http://ros.org/wiki/xacro">
+    <!-- Data Sheet:
+            https://www.zivid.com/hubfs/Zivid%20One%20Plus%20Datasheet%20(1).pdf?hsCtaTracking=f6b119a4-7444-47ac-83a3-44d4840aa429%7Ccabb4557-32f2-4851-9612-99fe7552235b
+    -->
+    <!-- Import Gazebo-Settings -->
+    <xacro:include filename="$(find zivid_description)/urdf/macros/zivid_one_plus_camera.gazebo.xacro" />
     <!-- Zivid One+ Types: Can be accessed globally and used as identifiers -->
     <xacro:property name="Zivid_One_Plus_S" value="0" scope="global" />
@@ -31,4 +36,9 @@
                 </geometry>
             </collision>
+            <!-- Inertial -->
+            <inertial>
+                <mass value="2"/>
+                <inertia ixx="0.0" ixy="0.0" ixz="0.0" iyy="0.0" iyz="0.0" izz="0.0"/>
+            </inertial>
         </link>
         <!-- Zivid Optical Frame (Measurement Frame)-->
@@ -50,4 +60,6 @@
             <child link="${prefix}_optical_frame"/>
         </joint>
+        <!--Extensions -->
+        <xacro:zivid_one_plus_gazebo prefix="${prefix}"/>
     </xacro:macro>
 </robot>

Commit message: Description for Zivid Two M70

File: zivid_description/urdf/macros/zivid_one_plus_camera.xacro (robot description, xacro)
@@ -18,5 +18,11 @@
         <color rgba="0.25 0.25 0.25 1"/>
     </material>
-    <xacro:macro name="zivid_one_plus_camera" params="prefix type">
+    <xacro:macro name="zivid_one_plus_camera" params="parent prefix type">
+        <!-- Joint to External Link -->
+        <joint name="${prefix}_base_link_joint" type="fixed">
+            <origin xyz="0.0 0.0 0.0" rpy="${0.0*pi} ${0.0*pi} ${0.0*pi}"/>
+            <parent link="${parent}"/>
+            <child link="${prefix}_base_link"/>
+        </joint>
         <!-- Zivid Base Link -->
         <link name="${prefix}_base_link">

File: zivid_description/urdf/zivid_one_plus_l_camera.urdf.xacro (robot description, xacro)
@@ -1,5 +1,6 @@
 <?xml version="1.0"?>
 <robot name="zivid_one_plus_camera_robot" xmlns:xacro="http://www.ros.org/wiki/xacro">
+    <link name="world"/>
     <xacro:include filename="$(find zivid_description)/urdf/macros/zivid_one_plus_camera.xacro"/>
-    <xacro:zivid_one_plus_camera prefix="zivid" type="${Zivid_One_Plus_L}"/>
+    <xacro:zivid_one_plus_camera parent="world" prefix="zivid" type="${Zivid_One_Plus_L}"/>
 </robot>

File: zivid_description/urdf/zivid_one_plus_m_camera.urdf.xacro (robot description, xacro)
@@ -1,5 +1,6 @@
 <?xml version="1.0"?>
 <robot name="zivid_one_plus_camera_robot" xmlns:xacro="http://www.ros.org/wiki/xacro">
+    <link name="world"/>
     <xacro:include filename="$(find zivid_description)/urdf/macros/zivid_one_plus_camera.xacro"/>
-    <xacro:zivid_one_plus_camera prefix="zivid" type="${Zivid_One_Plus_M}"/>
+    <xacro:zivid_one_plus_camera parent="world" prefix="zivid" type="${Zivid_One_Plus_M}"/>
 </robot>

File: zivid_description/urdf/zivid_one_plus_s_camera.urdf.xacro (robot description, xacro)
@@ -1,5 +1,6 @@
 <?xml version="1.0"?>
 <robot name="zivid_one_plus_camera_robot" xmlns:xacro="http://www.ros.org/wiki/xacro">
+    <link name="world"/>
     <xacro:include filename="$(find zivid_description)/urdf/macros/zivid_one_plus_camera.xacro"/>
-    <xacro:zivid_one_plus_camera prefix="zivid" type="${Zivid_One_Plus_S}"/>
+    <xacro:zivid_one_plus_camera parent="world" prefix="zivid" type="${Zivid_One_Plus_S}"/>
 </robot>
